File: Electronics/Optical Board/Optical Board.kicad_sch (KiCad schematic)
At the start: 10 parts, among them J2 OPTICAL

Commit message: Footprint changes
Parts:
- J2: footprint Connector_JST:JST_EH_S9B-EH_1x09_P2.50mm_Horizontal -> Connector_JST:JST_PH_S9B-PH-SM4-TB_1x09-1MP_P2.00mm_Horizontal
Connections:
- net +3V3: now also J2.4 (Pin_4); no longer J2.6 (Pin_6)
- net LED1: now also J2.3 (Pin_3); no longer J2.7 (Pin_7)
- net LED2: now also J2.2 (Pin_2); no longer J2.8 (Pin_8)
- net LED3: now also J2.1 (Pin_1); no longer J2.9 (Pin_9)
- net PD1: now also J2.9 (Pin_9); no longer J2.1 (Pin_1)
- net PD2: now also J2.8 (Pin_8); no longer J2.2 (Pin_2)
- net PD3: now also J2.7 (Pin_7); no longer J2.3 (Pin_3)
- net PD4: now also J2.6 (Pin_6); no longer J2.4 (Pin_4)
Changed lines of the file:
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@@
 		(lib_id "Connector_Generic:Conn_01x09")
 		(at 227.33 185.42 0)
+		(mirror x)
 		(unit 1)
 		(exclude_from_sim no)
@@
 		(on_board yes)
 		(dnp no)
-		(fields_autoplaced yes)
 		(property "Reference" "J2"
-			(at 229.87 184.1499 0)
+			(at 227.33 168.91 0)
 			(effects
 				(font
 					(size 1.27 1.27)
 				)
-				(justify left)
 			)
 		)
 		(property "Value" "OPTICAL"
-			(at 229.87 186.6899 0)
+			(at 227.33 171.45 0)
 			(effects
 				(font
 					(size 1.27 1.27)
 				)
-				(justify left)
 			)
 		)
-		(property "Footprint" "Connector_JST:JST_EH_S9B-EH_1x09_P2.50mm_Horizontal"
+		(property "Footprint" "Connector_JST:JST_PH_S9B-PH-SM4-TB_1x09-1MP_P2.00mm_Horizontal"
 			(at 227.33 185.42 0)
 			(effects
@@
 		)
 		(instances
-			(project "V1"
+			(project "Optical Board"
 				(path "/6465b793-86b5-4750-83bc-367c462e0283"
 					(reference "J2")
