File: Electronics/V1/V1.kicad_sch (KiCad schematic)
At the start: 45 parts, among them J1 BA9VPC, J3 GPIO, Q1 PMV41XPAR, Q3 PMV41XPAR, SW1 PVA1 EE H1 3.5N V2, U1 TPS7A4533, U2 TCA9517ADGK, U3 XIAO-ESP32-C3, U4 TPS72218, U5 ADPD1080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

Commit message: minor changes
Parts:
- added J2: OPTICAL, Connector_JST:JST_EH_S8B-EH_1x08_P2.50mm_Horizontal, symbol Connector_Generic:Conn_01x08
Connections:
- net +3V3: now also J2.5 (Pin_5)
- net LED2: now reaches LED1.3 (KGREEN), U5.24 (LEDX2)
- net LED2: now also J2.7 (Pin_7)
- net PD2: now reaches PD2.2 (A), U5.8 (PD2)
- net PD2: now also J2.2 (Pin_2)
- net LED3: now reaches LED1.4 (KRED), U5.25 (LEDX3)
- net LED3: now also J2.8 (Pin_8)
- net PD4: now reaches PD4.2 (A), U5.10 (PD4)
- net PD4: now also J2.4 (Pin_4)
- net LED1: now reaches LED1.1 (KIR), U5.23 (LEDX1)
- net LED1: now also J2.6 (Pin_6)
- net PD1: now reaches PD1.2 (A), U5.7 (PD1)
- net PD1: now also J2.1 (Pin_1)
- net PD3: now reaches PD3.2 (A), U5.9 (PD3)
- net PD3: now also J2.3 (Pin_3)

Commit message: Swapped I2C shifter for PCA9306DC
Parts:
- removed U2: TCA9517ADGK, Package_SO:VSSOP-8_3x3mm_P0.65mm, symbol Logic_LevelTranslator:TCA9517ADGK
- added J4: JST, Connector_JST:JST_PH_S2B-PH-K_1x02_P2.00mm_Horizontal, symbol Connector_Generic:Conn_01x02
- added R13, R14: 10k, Resistor_SMD:R_0603_1608Metric_Pad0.98x0.95mm_HandSolder, symbol Device:R
- added R15: 200K, Resistor_SMD:R_0603_1608Metric_Pad0.98x0.95mm_HandSolder, symbol Device:R
- added R16: 0, Resistor_SMD:R_0603_1608Metric_Pad0.98x0.95mm_HandSolder, symbol Device:R
- added U6: PCA9306DC, Package_SO:VSSOP-8_2.3x2mm_P0.5mm, symbol Interface:PCA9306DC
- J2: footprint Connector_JST:JST_EH_S8B-EH_1x08_P2.50mm_Horizontal -> Connector_JST:JST_PH_S8B-PH-K_1x08_P2.00mm_Horizontal
- R5: value changeme -> 200k
Connections:
- net +1V8: now also U6.2 (VREF1)
- net +3V3: now also R15.1; no longer C4.1
- net BAT+: now also J4.1 (Pin_1)
- net GND: now also J4.2 (Pin_2), U6.1 (GND)
- net PPG_SCL: now also U6.3 (SCL1)
- net PPG_SDA: now also U6.4 (SDA1)
- net UC_SCL: now also R13.2, U6.6 (SCL2)
- net UC_SDA: now also R14.2, U6.5 (SDA2)
- net I2C_EN: no longer names the net of U3.4 (D3)
- new net: C4.1, R13.1, R14.1, R15.2, R16.1, U6.7 (VREF2)
- new net: R16.2, U6.8 (EN)
- no-connect marks 4 -> 5
Other:
- note added: "EN should be pulled up for bi-directional data flow"
- note added: "GPIO Level shifter required for communication between OFE (1.8V) and Microcontroller (3.3V)"
- note added: "I2C Level shifter required for communication between OFE (1.8V) and Microcontroller (3.3V)"
- note added: "On-off push switch controlled FET"
- note removed: "Choose a pull down"
- note removed: "gpio Level shifter required for communication between OFE (1.8V) and Microcontroller (3.3v)"
- note removed: "i2c Level shifter required for communication between OFE (1.8V) and Microcontroller (3.3v)"
- moved on the sheet: C3, C4, D1, J1, J3, Q3, R1, R11, R12, R2, SW1

Commit message: Changing from integrated optical sensors to separate PCB
Parts:
- removed R13, R14: 10k, Resistor_SMD:R_0603_1608Metric_Pad0.98x0.95mm_HandSolder, symbol Device:R
- J2: footprint Connector_JST:JST_PH_S8B-PH-K_1x08_P2.00mm_Horizontal -> Connector_JST:JST_EH_S9B-EH_1x09_P2.50mm_Horizontal; symbol Connector_Generic:Conn_01x08 -> Connector_Generic:Conn_01x09
- J4: footprint Connector_JST:JST_PH_S2B-PH-K_1x02_P2.00mm_Horizontal -> Connector_JST:JST_EH_S2B-EH_1x02_P2.50mm_Horizontal
Connections:
- net +3V3: now also J2.6 (Pin_6); no longer J2.5 (Pin_5)
- net LED1: now also J2.7 (Pin_7); no longer J2.6 (Pin_6)
- net LED2: now also J2.8 (Pin_8); no longer J2.7 (Pin_7)
- net LED3: now also J2.9 (Pin_9); no longer J2.8 (Pin_8)
- net PD_K: now also J2.5 (Pin_5)

Commit message: Footprint changes
Parts:
- J2: footprint Connector_JST:JST_EH_S9B-EH_1x09_P2.50mm_Horizontal -> Connector_JST:JST_PH_S9B-PH-SM4-TB_1x09-1MP_P2.00mm_Horizontal
- J4: footprint Connector_JST:JST_EH_S2B-EH_1x02_P2.50mm_Horizontal -> Connector_JST:JST_PH_S2B-PH-SM4-TB_1x02-1MP_P2.00mm_Horizontal
- U5: footprint Package_CSP:LFCSP-28-1EP_5x5mm_P0.5mm_EP3.14x3.14mm -> CUSTOM:ADPD1080
Connections:
- net +3V3: now also J2.4 (Pin_4); no longer J2.6 (Pin_6)
- net LED1: now also J2.3 (Pin_3); no longer J2.7 (Pin_7)
- net LED2: now also J2.2 (Pin_2); no longer J2.8 (Pin_8)
- net LED3: now also J2.1 (Pin_1); no longer J2.9 (Pin_9)
- net PD1: now also J2.9 (Pin_9); no longer J2.1 (Pin_1)
- net PD2: now also J2.8 (Pin_8); no longer J2.2 (Pin_2)
- net PD3: now also J2.7 (Pin_7); no longer J2.3 (Pin_3)
- net PD4: now also J2.6 (Pin_6); no longer J2.4 (Pin_4)
Changed lines of the file:
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@@
 			)
 		)
-		(property "Footprint" "Package_CSP:LFCSP-28-1EP_5x5mm_P0.5mm_EP3.14x3.14mm"
+		(property "Footprint" "CUSTOM:ADPD1080"
 			(at 228.6 226.06 0)
 			(effects
@@
 		(lib_id "Connector_Generic:Conn_01x09")
 		(at 360.68 175.26 0)
-		(unit 1)
-		(exclude_from_sim no)
-		(in_bom yes)
-		(on_board yes)
-		(dnp no)
-		(fields_autoplaced yes)
+		(mirror x)
+		(unit 1)
+		(exclude_from_sim no)
+		(in_bom yes)
+		(on_board yes)
+		(dnp no)
 		(property "Reference" "J2"
-			(at 363.22 173.9899 0)
-			(effects
-				(font
-					(size 1.27 1.27)
-				)
-				(justify left)
+			(at 360.68 158.75 0)
+			(effects
+				(font
+					(size 1.27 1.27)
+				)
 			)
 		)
 		(property "Value" "OPTICAL"
-			(at 363.22 176.5299 0)
-			(effects
-				(font
-					(size 1.27 1.27)
-				)
-				(justify left)
-			)
-		)
-		(property "Footprint" "Connector_JST:JST_EH_S9B-EH_1x09_P2.50mm_Horizontal"
+			(at 360.68 161.29 0)
+			(effects
+				(font
+					(size 1.27 1.27)
+				)
+			)
+		)
+		(property "Footprint" "Connector_JST:JST_PH_S9B-PH-SM4-TB_1x09-1MP_P2.00mm_Horizontal"
 			(at 360.68 175.26 0)
 			(effects
@@
 			)
 		)
-		(property "Footprint" "Connector_JST:JST_EH_S2B-EH_1x02_P2.50mm_Horizontal"
+		(property "Footprint" "Connector_JST:JST_PH_S2B-PH-SM4-TB_1x02-1MP_P2.00mm_Horizontal"
 			(at 38.862 98.552 0)
 			(effects
